Commit message: Added base_footprint link to URDF

File: go1_description/xacro/robot.xacro (robot description, xacro)
@@ -30,4 +30,12 @@
         </visual>
     </link>
+    <link name="base_footprint" />
+      <joint name="base_to_footprint" type="prismatic">
+             <parent link="base"/>
+             <child link="base_footprint"/>
+             <origin xyz = "0 0 0" rpy="0 0 0"/>
+             <axis xyz="0 0 1" />
+             <limit effort="100000.0" lower="-1.0" upper="0.0" velocity="100000.0"/>
+     </joint>
     <joint name="floating_base" type="fixed">
         <origin rpy="0 0 0" xyz="0 0 0"/>

Commit message: Made base_footprint link optional

File: go1_description/xacro/robot.xacro (robot description, xacro)
@@ -2,4 +2,5 @@
 <robot name="go1" xmlns:xacro="http://www.ros.org/wiki/xacro">
     <xacro:arg name="DEBUG" default="false"/>
+    <xacro:arg name="enable_base_footprint" default="false"/>
     <xacro:include filename="$(find go1_description)/xacro/const.xacro"/>
     <xacro:include filename="$(find go1_description)/xacro/materials.xacro"/>
@@ -30,12 +31,14 @@
         </visual>
     </link>
-    <link name="base_footprint" />
-      <joint name="base_to_footprint" type="prismatic">
-             <parent link="base"/>
-             <child link="base_footprint"/>
-             <origin xyz = "0 0 0" rpy="0 0 0"/>
-             <axis xyz="0 0 1" />
-             <limit effort="100000.0" lower="-1.0" upper="0.0" velocity="100000.0"/>
-     </joint>
+    <xacro:if value="$(arg enable_base_footprint)">
+        <link name="base_footprint" />
+        <joint name="base_to_footprint" type="prismatic">
+                <parent link="base"/>
+                <child link="base_footprint"/>
+                <origin xyz = "0 0 0" rpy="0 0 0"/>
+                <axis xyz="0 0 1" />
+                <limit effort="100000.0" lower="-1.0" upper="0.0" velocity="100000.0"/>
+        </joint>
+    </xacro:if>
     <joint name="floating_base" type="fixed">
         <origin rpy="0 0 0" xyz="0 0 0"/>

Commit message: Added base_link base_footprint and connections

File: go1_description/xacro/robot.xacro (robot description, xacro)
@@ -3,4 +3,5 @@
     <xacro:arg name="DEBUG" default="false"/>
     <xacro:arg name="enable_base_footprint" default="false"/>
+    <xacro:arg name="enable_lidar" default="false"/>
     <xacro:include filename="$(find go1_description)/xacro/const.xacro"/>
     <xacro:include filename="$(find go1_description)/xacro/materials.xacro"/>
@@ -41,4 +42,45 @@
         </joint>
     </xacro:if>
+    <!-- <xacro:if value="$(arg enable_lidar)"> -->
+        <!-- <link name="base_link">
+            <visual>
+                <origin rpy="0 0 0" xyz="0 0 0"/>
+                <geometry>
+                    <box size="0.001 0.001 0.001"/>
+                </geometry>
+            </visual>
+        </link>
+        <link name="base_footprint">
+            <visual>
+                <origin rpy="0 0 0" xyz="0 0 0"/>
+                <geometry>
+                    <box size="0.001 0.001 0.001"/>
+                </geometry>
+            </visual>
+        </link> -->
+        <!-- <link name="base_link" /> -->
+        <!-- <joint name="rslidar_to_base_link" type="fixed">
+                <parent link="rslidar"/>
+                <child link="base_link"/>
+                <origin xyz = "0 0 0" rpy="0 0 0"/>
+                <axis xyz="0 0 1" />
+                <limit effort="100000.0" lower="-1.0" upper="0.0" velocity="100000.0"/>
+        </joint>
+        <joint name="base_link_to_base" type="fixed">
+                <parent link="base_link"/>
+                <child link="base"/>
+                <origin xyz = "0 0 0" rpy="0 0 0"/>
+                <axis xyz="0 0 1" />
+                <limit effort="100000.0" lower="-1.0" upper="0.0" velocity="100000.0"/>
+        </joint> -->
+        <!-- <link name="base_footprint" /> -->
+        <!-- <joint name="base_link_to_base_footprint" type="fixed">
+                <parent link="base_link"/>
+                <child link="base_footprint"/>
+                <origin xyz = "0 0 1" rpy="0 0 0"/>
+                <axis xyz="0 0 1" />
+                <limit effort="100000.0" lower="-1.0" upper="0.0" velocity="100000.0"/>
+        </joint>
+    </xacro:if> -->
     <joint name="floating_base" type="fixed">
         <origin rpy="0 0 0" xyz="0 0 0"/>

Commit message: Updated high JSP and xacro to properly publish body height

File: go1_description/xacro/robot.xacro (robot description, xacro)
@@ -32,11 +32,18 @@
     </link>
     <xacro:if value="$(arg enable_base_footprint)">
+        <link name="height_measurement" />
+        <!-- Measured empirically from difference between actual and reported body height -->
+        <joint name="base_to_height" type="fixed">
+            <origin rpy="0 0 0" xyz="0 0 -0.015"/>
+            <parent link="base"/>
+            <child link="height_measurement"/>
+        </joint>
         <link name="base_footprint" />
-        <joint name="base_to_footprint" type="prismatic">
-                <parent link="base"/>
+        <joint name="height_to_footprint" type="prismatic">
+                <parent link="height_measurement"/>
                 <child link="base_footprint"/>
                 <origin xyz = "0 0 0" rpy="0 0 0"/>
-                <axis xyz="0 0 1" />
-                <limit effort="100000.0" lower="-1.0" upper="0.0" velocity="100000.0"/>
+                <axis xyz="0 0 -1" />
+                <limit effort="100000.0" lower="0.0" upper="1.0" velocity="100000.0"/>
         </joint>
     </xacro:if>

Commit message: Added Nav2 frame names to URDF and high launch files

File: go1_description/xacro/robot.xacro (robot description, xacro)
@@ -2,5 +2,5 @@
 <robot name="go1" xmlns:xacro="http://www.ros.org/wiki/xacro">
     <xacro:arg name="DEBUG" default="false"/>
-    <xacro:arg name="enable_base_footprint" default="false"/>
+    <xacro:arg name="use_nav2_links" default="false"/>
     <xacro:include filename="$(find go1_description)/xacro/const.xacro"/>
     <xacro:include filename="$(find go1_description)/xacro/materials.xacro"/>
@@ -31,10 +31,16 @@
         </visual>
     </link>
-    <xacro:if value="$(arg enable_base_footprint)">
+    <xacro:if value="$(arg use_nav2_links)">
+        <link name="base_link" />
+        <joint name="base_link_to_base" type="fixed">
+            <origin rpy="0 0 0" xyz="0 0 0"/>
+            <parent link="base_link"/>
+            <child link="base"/>
+        </joint>
         <link name="height_measurement" />
         <!-- Measured empirically from difference between actual and reported body height -->
-        <joint name="base_to_height" type="fixed">
+        <joint name="base_link_to_height" type="fixed">
             <origin rpy="0 0 0" xyz="0 0 -0.015"/>
-            <parent link="base"/>
+            <parent link="base_link"/>
             <child link="height_measurement"/>
         </joint>
@@ -46,4 +52,11 @@
                 <axis xyz="0 0 -1" />
                 <limit effort="100000.0" lower="0.0" upper="1.0" velocity="100000.0"/>
+        </joint>
+        <link name="base_laser" />
+        <joint name="base_link_to_lidar" type="fixed">
+            <!-- TODO need to measure mounting or make this a parameter -->
+            <origin rpy="0 0 0" xyz="0 0 0.17"/>
+            <parent link="base_link"/>
+            <child link="base_laser"/>
         </joint>
     </xacro:if>

Commit message: Updated lidar offsets to be parameters, defaults based on NU custom mount

File: go1_description/xacro/robot.xacro (robot description, xacro)
@@ -3,4 +3,7 @@
     <xacro:arg name="DEBUG" default="false"/>
     <xacro:arg name="use_nav2_links" default="false"/>
+    <xacro:arg name="lidar_x_offset" default="0.0525"/>
+    <xacro:arg name="lidar_y_offset" default="0.0"/>
+    <xacro:arg name="lidar_z_offset" default="0.21"/>
     <xacro:include filename="$(find go1_description)/xacro/const.xacro"/>
     <xacro:include filename="$(find go1_description)/xacro/materials.xacro"/>
@@ -56,5 +59,5 @@
         <joint name="base_link_to_lidar" type="fixed">
             <!-- TODO need to measure mounting or make this a parameter -->
-            <origin rpy="0 0 0" xyz="0 0 0.17"/>
+            <origin rpy="0 0 0" xyz="$(arg lidar_x_offset) $(arg lidar_y_offset) $(arg lidar_z_offset)"/>
             <parent link="base_link"/>
             <child link="base_laser"/>
